File: Main/P12_00_00-MainKiCad/P12_00_00-MainKiCad.kicad_sch (KiCad schematic)
At the start: 53 parts, among them K1 hk19f-dc5v-shg, Q1 2N3904

Commit message: KiCAD modifications
Parts:
- 5V1: renamed from 5V; footprint (none) -> MountingHole:MountingHole_2.1mm
- D1: footprint Diode_THT:D_DO-41_SOD81_P10.16mm_Horizontal -> Diode_THT:D_DO-34_SOD68_P7.62mm_Horizontal
- D2, D3, D4, D5, D6: renamed from D?; footprint Diode_THT:D_DO-41_SOD81_P10.16mm_Horizontal -> Diode_THT:D_DO-34_SOD68_P7.62mm_Horizontal
- GND1: renamed from GND; footprint (none) -> MountingHole:MountingHole_2.1mm
- GPIO_10, GPIO_11, GPIO_12, GPIO_13, GPIO_14, GPIO_9: footprint (none) -> MountingHole:MountingHole_2.1mm
- GPIO_4: renamed from GPIO_04; footprint (none) -> MountingHole:MountingHole_2.1mm
- GPIO_5: renamed from GPIO_05; footprint (none) -> MountingHole:MountingHole_2.1mm
- GPIO_6: renamed from GPIO_06; footprint (none) -> MountingHole:MountingHole_2.1mm
- GPIO_7: renamed from GPIO_07; footprint (none) -> MountingHole:MountingHole_2.1mm
- GPIO_8: renamed from GPIO_08; footprint (none) -> MountingHole:MountingHole_2.1mm
- L_COM1: renamed from L_COM; footprint (none) -> MountingHole:MountingHole_2.1mm
- L_LR1: renamed from L_LR; footprint (none) -> MountingHole:MountingHole_2.1mm
- R1, R10, R12, R13, R15, R2, R3, R4, R6, R7, R9: footprint (none) -> Resistor_THT:R_Axial_DIN0204_L3.6mm_D1.6mm_P5.08mm_Horizontal
- R11, R14, R16, R5, R8: renamed from R?; footprint (none) -> Resistor_THT:R_Axial_DIN0204_L3.6mm_D1.6mm_P5.08mm_Horizontal
- R_COM1: renamed from R_COM; footprint (none) -> MountingHole:MountingHole_2.1mm
- R_LR1: renamed from R_LR; footprint (none) -> MountingHole:MountingHole_2.1mm
- UD1: renamed from UD; footprint (none) -> MountingHole:MountingHole_2.1mm
- VCC1: renamed from VCC; footprint (none) -> MountingHole:MountingHole_2.1mm
- gave numbers to parts that had none: 10

Commit message: Working with the schematic
Parts:
- removed 5V1, GND1, GPIO_10, GPIO_11, GPIO_12, GPIO_13, GPIO_14, GPIO_4, GPIO_5, GPIO_6, GPIO_7, GPIO_8, GPIO_9, L_COM1, L_LR1, R_COM1, R_LR1, UD1, VCC1: L_COM, MountingHole:MountingHole_2.1mm, symbol Mechanical:MountingHole
- removed D1, D2, D3, D4, D6: 1N4002, Diode_THT:D_DO-34_SOD68_P7.62mm_Horizontal, symbol Diode:1N4002
- removed K4, K5, K6: hk19f-dc5v-shg, Relay_THT:Relay_DPDT_Schrack-RT2-FormC_RM5mm, symbol Relay:RT42xAxx
- removed Q2, Q5: 2N3904, Package_TO_SOT_THT:TO-92_Inline, symbol Transistor_BJT:2N3904
- added D11, D16: 1N4002, Diode_THT:D_DO-34_SOD68_P7.62mm_Horizontal, symbol Diode:1N4002
- added Mount1: 5V, MountingHole:MountingHole_2.1mm, symbol Mechanical:MountingHole
- added Mount10: A0, MountingHole:MountingHole_2.1mm, symbol Mechanical:MountingHole
- added Mount11: D00, MountingHole:MountingHole_2.1mm, symbol Mechanical:MountingHole
- added Mount12: D06, MountingHole:MountingHole_2.1mm, symbol Mechanical:MountingHole
- added Mount13: D07, MountingHole:MountingHole_2.1mm, symbol Mechanical:MountingHole
- added Mount14: A1, MountingHole:MountingHole_2.1mm, symbol Mechanical:MountingHole
- added Mount15: UD_OUT, MountingHole:MountingHole_2.1mm, symbol Mechanical:MountingHole
- added Mount16: UD_IN, MountingHole:MountingHole_2.1mm, symbol Mechanical:MountingHole
- added Mount17: R_RL_OUT, MountingHole:MountingHole_2.1mm, symbol Mechanical:MountingHole
- added Mount18: D08, MountingHole:MountingHole_2.1mm, symbol Mechanical:MountingHole
- added Mount19: R_RL_IN, MountingHole:MountingHole_2.1mm, symbol Mechanical:MountingHole
- added Mount2, Mount?: D03, MountingHole:MountingHole_2.1mm, symbol Mechanical:MountingHole
- added Mount20: D09, MountingHole:MountingHole_2.1mm, symbol Mechanical:MountingHole
- added Mount21: A2, MountingHole:MountingHole_2.1mm, symbol Mechanical:MountingHole
- added Mount22: D01, MountingHole:MountingHole_2.1mm, symbol Mechanical:MountingHole
- added Mount23: D10, MountingHole:MountingHole_2.1mm, symbol Mechanical:MountingHole
- added Mount24: D11, MountingHole:MountingHole_2.1mm, symbol Mechanical:MountingHole
- added Mount25: A3, MountingHole:MountingHole_2.1mm, symbol Mechanical:MountingHole
- added Mount26: R_COM_OUT, MountingHole:MountingHole_2.1mm, symbol Mechanical:MountingHole
- added Mount27: R_COM_IN, MountingHole:MountingHole_2.1mm, symbol Mechanical:MountingHole
- added Mount28: D12, MountingHole:MountingHole_2.1mm, symbol Mechanical:MountingHole
- added Mount29: GND, MountingHole:MountingHole_2.1mm, symbol Mechanical:MountingHole
- added Mount3: D13, MountingHole:MountingHole_2.1mm, symbol Mechanical:MountingHole
- added Mount30: 12V, MountingHole:MountingHole_2.1mm, symbol Mechanical:MountingHole
- added Mount31: D02, MountingHole:MountingHole_2.1mm, symbol Mechanical:MountingHole
- added Mount4: L_COM_Out, MountingHole:MountingHole_2.1mm, symbol Mechanical:MountingHole
- added Mount5: L_COM_IN, MountingHole:MountingHole_2.1mm, symbol Mechanical:MountingHole
- added Mount6: L_LR_OUT, MountingHole:MountingHole_2.1mm, symbol Mechanical:MountingHole
- added Mount7: D04, MountingHole:MountingHole_2.1mm, symbol Mechanical:MountingHole
- added Mount8: L_LR_IN, MountingHole:MountingHole_2.1mm, symbol Mechanical:MountingHole
- added Mount9: D05, MountingHole:MountingHole_2.1mm, symbol Mechanical:MountingHole
- added Q10, Q12, Q2, Q5, Q7, Q?: 2N3905, Package_TO_SOT_THT:TO-92_Inline_Wide, symbol Transistor_BJT:2N3905
- added Q11, Q13, Q8, Q9, Q?: 2N3904, Package_TO_SOT_THT:TO-92_Inline_Wide, symbol Transistor_BJT:2N3904
- added R17, R18, R19, R20, R21, R22, R23, R24, R25, R26, R27, R28, R? (x3): 220, Resistor_THT:R_Axial_DIN0204_L3.6mm_D1.6mm_P7.62mm_Horizontal, symbol Device:R
- Q1, Q3, Q4, Q6: footprint Package_TO_SOT_THT:TO-92_Inline -> Package_TO_SOT_THT:TO-92_Inline_Wide
- R1, R10, R13, R4, R7: value 2.2k -> 220; footprint Resistor_THT:R_Axial_DIN0204_L3.6mm_D1.6mm_P5.08mm_Horizontal -> Resistor_THT:R_Axial_DIN0204_L3.6mm_D1.6mm_P7.62mm_Horizontal
- R11, R14, R2, R5, R8: value 1k -> 220; footprint Resistor_THT:R_Axial_DIN0204_L3.6mm_D1.6mm_P5.08mm_Horizontal -> Resistor_THT:R_Axial_DIN0204_L3.6mm_D1.6mm_P7.62mm_Horizontal
- R12, R15, R16, R3, R6, R9: footprint Resistor_THT:R_Axial_DIN0204_L3.6mm_D1.6mm_P5.08mm_Horizontal -> Resistor_THT:R_Axial_DIN0204_L3.6mm_D1.6mm_P7.62mm_Horizontal
Connections:
- net at K2.A1: now also D5.1 (K), K1.A1, K3.A1, D11.1 (K), D16.1 (K)
- net at R1.2: no longer R2.1
- net at Q1.1 (E), Q3.1 (E), Q4.1 (E)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: now also R13.2, R8.1, Q11.1 (E), Q13.1 (E), Q8.1 (E), Q9.1 (E), R19.1, R24.2; no longer R11.2, R14.2, R5.2, R8.2
- net at D5.2 (A): now also K1.A2, Q4.3 (C)
- net at Q4.2 (B): now also R9.2; no longer R12.1
- net at R7.2: no longer R8.1
- net at Q1.3 (C): now also K1.24, Q2.3 (C); no longer K1.A1
- net at R4.1: now also R10.1, R15.1, Q10.1 (E), Q12.1 (E), Q2.1 (E), Q5.1 (E), Q7.1 (E), R21.1, R26.1; no longer K2.11
- net at K2.21: now also R14.1
- net at K2.24: now also Q6.3 (C), Q7.3 (C)
- net at R9.1: no longer Q3.2 (B)
- net at Q3.3 (C): now also K1.14, Q5.3 (C); no longer K3.A1
- net at K1.11: now also R6.2; no longer R1.1
- net at K1.21: now also R3.1
- net at Q1.2 (B): now also R1.1; no longer R3.1
- net at R3.2: now also R2.1
- net at R6.1: now also R8.2
- net at R13.1: now also R14.2
- net at K3.11: no longer R7.1
- net at R10.2, R11.1: now also Q5.2 (B)
- net at R4.2, R5.1: now also Q2.2 (B)
- net at R16.1: now also R15.2, Q7.2 (B); no longer Q6.2 (B)
- net at K3.21: now also R25.1
- net at K3.24: now also Q11.3 (C), Q12.3 (C)
- new net: Q10.2 (B), R21.2, R22.1
- new net: R17.1, R19.2
- new net: K2.11, R17.2
- new net: Q13.2 (B), R28.2
- new net: K2.14, Q10.3 (C), Q8.3 (C)
- new net: D11.2 (A), K2.A2, Q9.3 (C)
- new net: D16.2 (A), K3.A2, Q13.3 (C)
- new net: Q?.2 (B), R?.1
- new net: Q?.1 (E), R?.1
- new net: Q?.2 (B), R?.1, R?.2
- new net: Q11.2 (B), R23.1
- new net: Q12.2 (B), R26.2, R27.1
- new net: R24.1, R25.2
- new net: Q6.2 (B), R12.1
- new net: Q3.2 (B), R7.1
- new net: Q?.3 (C), Q?.3 (C)
- new net: Q8.2 (B), R18.1
- new net: Q9.2 (B), R20.2
- now unconnected: K1.12, K2.12, K3.12, K3.14
